File: circuit_designs/PCBs/Final_Versions/CanSat_Power_Management_Board/CanSat_Power_Management_Board.kicad_pcb (KiCad board)
At the start: 4 copper layers, 95 x 95 mm, 63 parts, among them J1 MCU Switch (7.4V), J2 7.4V Battery, J3 Sensor Board, J4 Booster Switch (3.7V), J5 3.7V Battery, Q1 BS170, Q2 BSS84, U1 LM2596T-ADJ, U3 NE555P

Commit message: PCB improvements for the future
Parts:
- removed the G*** at (120.8, 123.0)
- added G***: LOGO, Graphics:uoft_text_2, B.Cu at (147.8, 141.8)
- added G***: LOGO, Graphics:uoft_coat_of_arms_2, B.Cu at (157.2, 140.8)
- added G***: LOGO, Graphics:logo, B.Cu at (123.5, 124.0)
- added G***: LOGO, Graphics:rsx_logo_2, B.Cu at (180.8, 123.2)
- moved TP5 2.50 mm to (116.0, 114.8)
- moved G*** 0.79 mm to (123.0, 121.0)
- moved G*** 0.50 mm to (117.8, 106.2)
Routing:
- net ADC: track 94.7 -> 89.6 mm
- net 7.4V: track 211.3 -> 207.9 mm
- net 3.3V: track 55.2 -> 54.2 mm
Other:
- board text added: "Booster Circuit"
- board text added: "LM2596T-ADJ"
